File: mcp3008_rpi_SOIP.sch (EAGLE design)
At the start: 10 parts

Commit message: i2c board complete
Parts:
- removed JP1, JP2: (no value), pinhead:PINHD-1X2
- removed U$4, U$5, U$6, U$7: ICUBE_I2C, jt_lib:ICUBE_I2C
- U$3: value MCP3008P -> MCP3008SL; device MCP3008:MCP3008P -> MCP3008:MCP3008SL
Connections:
- removed net N$13: JP1.2, U$2.GPIO23
- removed net N$14: U$2.GPIO1_SCL0, U$4.P$3_SCL, U$5.P$3_SCL, U$6.P$3_SCL, U$7.P$3_SCL
- removed net N$15: U$2.GPIO0_SDA0, U$4.P$2_SDA, U$5.P$2_SDA, U$6.P$2_SDA, U$7.P$2_SDA
- removed net N$16: JP2.2, U$2.GPIO24
- net GND: no longer JP1.1, JP2.1, U$4.P$4_GND, U$5.P$4_GND, U$6.P$4_GND, U$7.P$4_GND
- net N$12: no longer U$5.P$1_VCC, U$6.P$1_VCC, U$7.P$1_VCC
- net VCC: now also U$2.5V_0; no longer U$2.3V3_0, U$4.P$1_VCC
